File: kicad/usb3-hub.kicad_pcb (KiCad board)
At the start: 6 copper layers, 70 x 140 mm, 229 parts, among them J1001 USB3_A, J101 DISPLAY, J102 USB3_B_Micro, J103 Barrel_Jack_Switch, J301 Debug, J302 Conn_01x03_Pin, J303 Conn_01x05_Pin, J501 USB3_A, J601 USB3_A, J701 USB3_A, J801 USB3_A, J901 USB3_A, Q303 2N7002, SW1001 SW_Push, SW301 SW_Push, SW501 SW_Push, SW601 SW_Push, SW701 SW_Push, SW801 SW_Push, SW901 SW_Push, U1001 AP22804AW5, U201 USB5807, U301 W25Q16JVSS, U302 RP2040, U303 AP22804AW5, U401 TLV1117-33, U402 AP62250Z6, U501 INA381A1, U502 AP22804AW5, U601 INA381A1, U602 AP22804AW5, U701 INA381A1, U702 AP22804AW5, U801 AP22804AW5, U901 AP22804AW5, Y201 25Mhz, Y301 12Mhz

Commit message: Some more routing
Parts:
- moved C407 0.82 mm to (156.7, 85.9)
- moved C406 0.80 mm to (156.7, 88.0)
- moved R403 0.70 mm to (164.5, 86.0)
Routing:
- net /Hub/Port1.PRT_CTRL: track 2.91 -> 86.1 mm, vias 1 -> 4
- net GND: track 114.7 -> 164.8 mm, vias 74 -> 107
- net +5V: track 3.37 -> 37.6 mm, vias 0 -> 7
- net /Port1/Shield: track 0.00 -> 27.5 mm
- net /Port6/Shield: track 0.00 -> 27.2 mm
- net /Port4/Shield: track 0.00 -> 27.2 mm
- net /Port2/Shield: track 0.00 -> 27.0 mm
- net /Port3/Shield: track 0.00 -> 26.7 mm
- net /Port5/Shield: track 5.02 -> 27.2 mm
- net +3V3: track 92.5 -> 105.3 mm, vias 26 -> 35
- net /Port1/VBUS: track 12.3 -> 20.8 mm
- net /Port3/VBUS: track 13.5 -> 22.0 mm
- net /Port2/VBUS: track 13.2 -> 21.7 mm
- net /Port6/VBUS: track 0.00 -> 8.16 mm
- net /Port4/VBUS: track 0.00 -> 8.16 mm
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- added copper zone on F.Cu, net +1V2
- added copper zone on F.Cu, net +3V3
- added copper zone on F.Cu, net +5V
